File: pcbs/main_board/wheelberry_main/wheelberry_main.kicad_pcb (KiCad board)
At the start: 2 copper layers, 200 x 110 mm, 106 parts, among them J1 Conn_01x02_Male, J10 AudioJack3, J11 DIN-7, J2 USB_A, J3 USB_A, J4 DIN-7, J5 AudioJack2, J6 AudioJack3, J7 AudioJack2, J8 AudioJack2, J9 AudioJack3, P1 Conn_02x20_Odd_Even, Q1 Q_NMOS_DGS, U1 THN_15-2411, U2 ADS1115IDGS, U3 TLP222A-2, U4 MCP23017_SO, U5 MCP23017_SO, U6 TLP222A-2, U7 TLP222A-2, U8 TLP222A-2, U9 TLP222A-2

Commit message: v1.2
Parts:
- C1, C2: footprint Capacitor_THT:CP_Radial_D8.0mm_P5.00mm -> Capacitor_THT:CP_Radial_Tantal_D5.5mm_P5.00mm
- moved C20 19.2 mm to (231.8, 120.9)
- moved R24 16.0 mm to (85.6, 150.6), turned to 90 degrees
- moved R3 15.8 mm to (177.5, 130.3), turned to 180 degrees
- moved FB1 15.8 mm to (239.2, 121.9), turned to 270 degrees
- moved R6 14.3 mm to (166.1, 142.5), turned to 270 degrees
- moved C2 14.3 mm to (169.9, 130.3), turned to 180 degrees
- moved C1 12.3 mm to (190.9, 129.8)
- moved J2 10.8 mm to (191.5, 135.4)
- moved J3 6.91 mm to (172.7, 135.4), turned to 0 degrees
- moved R2 6.19 mm to (185.9, 142.7)
- moved D1 5.28 mm to (236.0, 130.3)
- moved J9 4.86 mm to (90.8, 118.3)
- moved R20 4.57 mm to (85.6, 144.0)
- moved C21 4.44 mm to (215.9, 122.7)
- moved R31 4.19 mm to (162.5, 155.9), turned to 90 degrees
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Routing:
- net Net-(Q1-Pad1): track 27.2 -> 48.0 mm, vias 0 -> 1
- net Net-(J3-Pad2): track 17.0 -> 5.17 mm
- net Net-(J3-Pad3): track 16.8 -> 5.22 mm
- net Net-(J9-PadS): track 35.3 -> 25.4 mm
- net Net-(J2-Pad3): track 15.4 -> 5.78 mm
- net Net-(J2-Pad2): track 15.0 -> 5.56 mm
- net Net-(J9-PadT): track 18.0 -> 27.4 mm
- net Net-(J11-Pad1): track 21.0 -> 11.6 mm
- net Net-(J11-Pad2): track 33.4 -> 23.9 mm
- net Net-(J4-Pad2): track 5.70 -> 14.2 mm
- net Net-(J4-Pad6): track 7.00 -> 15.2 mm
- net Net-(R20-Pad2): track 48.4 -> 40.4 mm
- net Net-(R24-Pad2): track 43.0 -> 35.9 mm
- net Net-(D1-Pad1): track 19.0 -> 12.6 mm
- net /Wheelberry Power/24V_IN: track 62.5 -> 68.0 mm
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Other:
- board text added: "Wheelberry 1.2"
- board text added: "c Darwin Innovation Ltd"
- board text removed: "Wheelberry 1.1"
