File: pcbs/main_board/wheelberry_main/wheelberry_power.sch (KiCad schematic (older format))
At the start: 29 parts, among them J2 USB_A, J3 USB_A, Q1 Q_NMOS_DGS, U1 THN_15-2411, U2 ADS1115IDGS

Commit message: v1.2
Parts:
- C1, C2: footprint Capacitor_THT:CP_Radial_D8.0mm_P5.00mm -> Capacitor_THT:CP_Radial_Tantal_D5.5mm_P5.00mm
Changed lines of the file:
@@
 F 0 "C1" H 1618 4646 50  0000 L CNN
 F 1 "47u" H 1618 4555 50  0000 L CNN
-F 2 "Capacitor_THT:CP_Radial_D8.0mm_P5.00mm" H 1538 4450 50  0001 C CNN
+F 2 "Capacitor_THT:CP_Radial_Tantal_D5.5mm_P5.00mm" H 1538 4450 50  0001 C CNN
 F 3 "~" H 1500 4600 50  0001 C CNN
 	1    1500 4600
@@
 F 0 "C2" H 3168 4646 50  0000 L CNN
 F 1 "47u" H 3168 4555 50  0000 L CNN
-F 2 "Capacitor_THT:CP_Radial_D8.0mm_P5.00mm" H 3088 4450 50  0001 C CNN
+F 2 "Capacitor_THT:CP_Radial_Tantal_D5.5mm_P5.00mm" H 3088 4450 50  0001 C CNN
 F 3 "~" H 3050 4600 50  0001 C CNN
 	1    3050 4600
